File: pcb/lattice-row-nine/lattice-row-nine.kicad_pcb (KiCad board)
At the start: 4 copper layers, 90.2 x 10.5 mm, 52 parts, among them J1 Conn_ARM_SWD_TagConnect_TC203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, J2 USB_C_Receptacle_USB2.0_16P, U1 STM32G431KBUx, U10 LPS22HH, U11 LPS22HH, U12 LPS22HH, U13 LPS22HH, U2 AMS1117-3.3, U3 SRV05-4, U4 LPS22HH, U5 LPS22HH, U6 LPS22HH, U7 LPS22HH, U8 LPS22HH, U9 LPS22HH, Y1 16MHz

Commit message: Final production
Other:
- board text added: "Designed By: Miguel Flores-Acton"
- board text added: "LatticeRow V1.0"
Changed lines of the file:
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@@
+			)
+		)
+		(property "LCSC" "C1341901"
+			(at 0 0 0)
+			(unlocked yes)
+			(layer "B.Fab")
+			(hide yes)
+			(effects
+				(font
+					(size 1 1)
+					(thickness 0.15)
+				)
+				(justify mirror)
 			)
 		)
@@
 		(layer "Edge.Cuts")
 	)
+	(gr_text "LatticeRow V1.0"
+		(at 111.5 81.25 0)
+		(layer "B.SilkS")
+		(effects
+			(font
+				(size 2 2)
+				(thickness 0.2)
+			)
+			(justify left bottom mirror)
+		)
+	)
+	(gr_text "Designed By: Miguel Flores-Acton"
+		(at 141.25 80.75 0)
+		(layer "B.SilkS")
+		(effects
+			(font
+				(size 1 1)
+				(thickness 0.1)
+			)
+			(justify left bottom mirror)
+		)
+	)
 	(segment
