File: pcb/sense-ring/sense-ring.kicad_sch (KiCad schematic)
At the start: 32 parts, among them J1 Conn_ARM_SWD_TagConnect_TC203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, J2 Conn_01x04_MountingPin, J3 Conn_01x04_MountingPin, U1 TJA1044GTK/3, U10 STM32G431KBUx, U11 NCP176, U9 ICM-42688-P, Y1 16MHz

Commit message: Layout sizing
Parts:
- C17, C18, C19: footprint (none) -> Capacitor_SMD:C_0402_1005Metric
Connections:
- net CLK is gone; now on net SCK: U9.13 (CLK)
- now unconnected: U9.10 (RESV), U9.2 (RESV), U9.3 (RESV)
Other:
- moved on the sheet: J3

Commit message: Save progress on sense-ring
Parts:
- removed C24: 100n, Capacitor_SMD:C_0402_1005Metric, symbol Device:C
- removed R2: 10k, Resistor_SMD:R_0402_1005Metric, symbol Device:R
Connections:
- net CS7: no longer U9.12 (CS)
- net RST: no longer U10.4 (PG10)
- net BOOT0: no longer names the net of U10.31 (PB8)
- new net CS8: U9.12 (CS)

Commit message: Initial layout
Parts:
- added C24, C30: 100n, Capacitor_SMD:C_0402_1005Metric, symbol Device:C
Connections:
- net +3V3: now also C24.1
- net +5V: now also C30.1
- net GND: now also C24.2, C30.2
- net XTALI: now also R3.2; no longer C25.2, Y1.1
- net XTALO: now also C25.2, Y1.1; no longer R3.2
Other:
- moved on the sheet: C28, C29, U11

Commit message: Finish sense-ring
Parts:
- C17: value 10n -> 100n; LCSC (none) -> C1525
- C18: LCSC (none) -> C1525
- C19: LCSC (none) -> C12530
- C28: footprint Capacitor_SMD:C_0603_1608Metric -> Capacitor_SMD:C_0402_1005Metric
Connections:
- net CNRX: now also U10.21 (PA11)
- net CNTX: now also U10.22 (PA12)
- net CS1: now also U10.7 (PA2)
- net CS2: now also U10.6 (PA1)
- net CS3: now also U10.30 (PB7)
- net CS4: now also U10.29 (PB6)
- net CS5: now also U10.31 (PB8)
- net CS6: now also U10.9 (PA4)
- net CS7: now also U10.13 (PB0)
- net CS8: now also U10.8 (PA3)
- net XTALI: now also C25.2, Y1.1; no longer R3.2
- net XTALO: now also R3.2; no longer C25.2, Y1.1
- net RST: no longer names the net of J1.3 (~{RESET})
- no-connect marks 2 -> 11
Other:
- moved on the sheet: C20, C21, C22, C23, U10
